File: corne-chocolate/v3/pcb/corne-chocolate.kicad_pcb (KiCad board)
At the start: 2 copper layers, 275.5 x 105.6 mm, 172 parts, among them J1 MJ-4PP-9, J2 OLED, J3 MJ-4PP-9, J4 OLED, SW1 SW_PUSH, SW10 SW_PUSH, SW11 SW_PUSH, SW12 SW_PUSH, SW13 SW_PUSH, SW14 SW_PUSH, SW15 SW_PUSH, SW16 SW_PUSH, SW17 SW_PUSH, SW18 SW_PUSH, SW19 SW_PUSH, SW2 SW_PUSH, SW20 SW_PUSH, SW21 SW_PUSH, SW22 SW_PUSH, SW23 SW_PUSH, SW24 SW_PUSH, SW25 SW_PUSH, SW26 SW_PUSH, SW27 SW_PUSH, SW28 SW_PUSH, SW29 SW_PUSH, SW3 SW_PUSH, SW30 SW_PUSH, SW31 SW_PUSH, SW32 SW_PUSH, SW33 SW_PUSH, SW34 SW_PUSH, SW35 SW_PUSH, SW36 SW_PUSH, SW37 SW_PUSH, SW38 SW_PUSH, SW39 SW_PUSH, SW4 SW_PUSH, SW40 SW_PUSH, SW41 SW_PUSH, SW42 SW_PUSH, SW5 SW_PUSH, SW6 SW_PUSH, SW7 SW_PUSH, SW8 SW_PUSH, SW9 SW_PUSH, U1 ProMicro, U2 ProMicro

Commit message: Add WIP 5-column PCB
Parts:
- removed D1, D13, D22, D28, D34, D7: D, kbd:D3_SMD_v2
- removed LED13, LED19, LED34, LED40, LED46, LED7: YS-SK6812MINI-E, kbd:YS-SK6812MINI-E
- removed SW1, SW13, SW22, SW28, SW34, SW7: SW_PUSH, custom_kicad:PG1350_socket_clean
Routing:
- net col0_r: track 177.9 -> 0.04 mm, vias 7 -> 0
- net col0: track 154.0 -> 0.00 mm, vias 3 -> 0
- net VCC: track 520.4 -> 427.1 mm, vias 41 -> 37
- net GND: track 586.5 -> 507.1 mm, vias 38 -> 35
- net VDD: track 550.3 -> 488.3 mm, vias 42 -> 38
- net GNDA: track 546.2 -> 492.8 mm, vias 32 -> 31
- net Net-(LED7-Pad4): track 28.1 -> 0.00 mm, vias 2 -> 0
- net row2: track 155.4 -> 131.3 mm
- net row2_r: track 156.6 -> 132.7 mm
- net row0_r: track 144.8 -> 121.0 mm
- net Net-(LED13-Pad4): track 23.5 -> 0.00 mm, vias 2 -> 0
- net row1_r: track 140.6 -> 117.1 mm
- net row1: track 136.3 -> 113.0 mm
- net row0: track 139.2 -> 115.9 mm
- net Net-(LED13-Pad2): track 23.0 -> 0.00 mm, vias 2 -> 0
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